File: board/board.kicad_pcb (KiCad board)
At the start: 2 copper layers, 21 x 13 mm, 1 part

Commit message: initial
Parts:
- added C1: 22pF, Capacitor_SMD:C_0603_1608Metric, F.Cu at (149.3, 91.8)
- added C2: 22pF, Capacitor_SMD:C_0603_1608Metric, F.Cu at (155.2, 93.0)
- added C3: 1uF, Capacitor_SMD:C_0603_1608Metric, F.Cu at (146.2, 98.2)
- added C4: 100nF, Capacitor_SMD:C_0603_1608Metric, F.Cu at (146.2, 101.2)
- added J1: 002_SPI, on_edge:on_edge_2x05_device, F.Cu at (140.0, 96.5)
- added J2: 012_CAN, on_edge:on_edge_2x05_host, F.Cu at (161.0, 96.5)
- added R1: 0R, Resistor_SMD:R_0603_1608Metric, F.Cu at (146.2, 95.2)
- added U1: MCP2517FD-xSL, Package_SO:SOIC-14_3.9x8.7mm_P1.27mm, F.Cu at (150.7, 98.2)
- added Y1: 20MhZ, Crystal:Crystal_SMD_Abracon_ABM8G-4Pin_3.2x2.5mm, F.Cu at (152.2, 91.8)
- LOGO1: moved to B.Cu
- moved LOGO1 0.30 mm to (150.3, 99.0), turned to 180 degrees
Routing:
- net /implementation/VDD: track 0.00 -> 25.3 mm, vias 0 -> 2
- net GND: track 0.00 -> 19.4 mm, vias 0 -> 15
- net Net-(J1-Pad10): track 0.00 -> 17.9 mm
- net /implementation/CS: track 0.00 -> 14.7 mm, vias 0 -> 1
- net /implementation/INT: track 0.00 -> 12.4 mm
- net /implementation/MOSI: track 0.00 -> 11.2 mm
- net /implementation/MISO: track 0.00 -> 11.1 mm, vias 0 -> 2
- net /implementation/CAN_TX: track 0.00 -> 10.1 mm
- net /implementation/CAN_RX: track 0.00 -> 10.1 mm
- net Net-(C2-Pad1): track 0.00 -> 8.19 mm
- net Net-(C1-Pad1): track 0.00 -> 7.11 mm
- net /implementation/CLK: track 0.00 -> 6.62 mm
- net /implementation/INT0: track 0.00 -> 6.56 mm, vias 0 -> 1
- net Net-(J1-Pad8): track 0.00 -> 3.96 mm, vias 0 -> 1
- net /implementation/INT1: track 0.00 -> 2.04 mm
- added copper zone on B.Cu, net GND
- added copper zone on F.Cu, net GND
Other:
- outline, holes or cut-outs redrawn
- board text added: "osf.002"
- board text added: "osf.012"
- board text added: "osf.b065.v1.0"
