File: board/implementation.kicad_sch (KiCad schematic)
At the start: 0 parts

Commit message: initial
Parts:
- added C1, C2: 22pF, Capacitor_SMD:C_0603_1608Metric, symbol Device:C_Small
- added C3: 1uF, Capacitor_SMD:C_0603_1608Metric, symbol Device:C_Small
- added C4: 100nF, Capacitor_SMD:C_0603_1608Metric, symbol Device:C_Small
- added U1: MCP2517FD-xSL, Package_SO:SOIC-14_3.9x8.7mm_P1.27mm, symbol Interface_CAN_LIN:MCP2517FD-xSL
- added Y1: 20MhZ, Crystal:Crystal_SMD_Abracon_ABM8G-4Pin_3.2x2.5mm, symbol Device:Crystal_GND24_Small
Connections:
- net GND: now also C1.2, C2.2, C3.2, C4.2, U1.7 (VSS), Y1.2, Y1.4
- new net: C1.1, U1.5 (OSC2), Y1.1
- new net: C2.1, U1.6 (OSC1), Y1.3
- new net CAN_RX: U1.1 (TXCAN)
- new net CAN_TX: U1.2 (RXCAN)
- new net CLK: U1.10 (SCK)
- new net CS: U1.13 (nCS)
- new net INT: U1.4 (~{INT})
- new net INT0: U1.9 (~{INT0}/GPIO0/XSTBY)
- new net INT1: U1.8 (~{INT1}/GPIO1)
- new net MISO: U1.12 (SDO)
- new net MOSI: U1.11 (SDI)
- new net VDD: C3.1, C4.1, U1.14 (VDD)
- no-connect marks 0 -> 1
